Commit message: add controller for wheeled robot

File: data/robots/fourwheels.urdf (robot description, URDF)
Before this commit: robot four_wheels, 5 links, 4 joints
Links:
- link chassis: mass 1 -> 20
Joints:
- joint chassis_wheel_fl: origin xyz=1 -1.5 0 rpy=1.57 0 0 -> xyz=1 1.5 0 rpy=1.57 0 0
- joint chassis_wheel_fr: origin xyz=1 1.5 0 rpy=1.57 0 0 -> xyz=1 -1.5 0 rpy=1.57 0 0
- joint chassis_wheel_rl: origin xyz=-1 -1.5 0 rpy=1.57 0 0 -> xyz=-1 1.5 0 rpy=1.57 0 0
- joint chassis_wheel_rr: origin xyz=-1 1.5 0 rpy=1.57 0 0 -> xyz=-1 -1.5 0 rpy=1.57 0 0

Commit message: use default desturtor

File: data/robots/fourwheels.urdf (robot description, URDF)
Before this commit: robot four_wheels, 5 links, 4 joints
Links:
- link chassis: geometry collision box size=3 2 0.5; visual box size=3 2 0.5
